Commit message: Oppdatering

File: urdf/robot_control.gazebo.xacro (robot description, xacro)
@@ -36,4 +36,49 @@
             <state_interface name="effort"/>
         </joint>
+        <joint name="arm_base_joint">
+            <command_interface name="position">
+                <param name="min">-${pi}</param>
+                <param name="max">${pi}</param>
+            </command_interface>
+            <state_interface name="position"/>
+            <state_interface name="velocity"/>
+            <state_interface name="effort"/>
+        </joint>
+        <joint name="link_1_joint">
+            <command_interface name="position">
+                <param name="min">-${pi/2}</param>
+                <param name="max">${pi/2}</param>
+            </command_interface>
+            <state_interface name="position"/>
+            <state_interface name="velocity"/>
+            <state_interface name="effort"/>
+        </joint>
+        <joint name="link_2_joint">
+            <command_interface name="position">
+                <param name="min">-${pi/2}</param>
+                <param name="max">${pi/2}</param>
+            </command_interface>
+            <state_interface name="position"/>
+            <state_interface name="velocity"/>
+            <state_interface name="effort"/>
+        </joint>
+        <joint name="link_3_joint">
+            <command_interface name="position">
+                <param name="min">-${pi/2}</param>
+                <param name="max">${pi/2}</param>
+            </command_interface>
+            <state_interface name="position"/>
+            <state_interface name="velocity"/>
+            <state_interface name="effort"/>
+        </joint>
+        <joint name="gripper_base_joint">
+            <command_interface name="position">
+                <param name="min">-${pi/2}</param>
+                <param name="max">${pi/2}</param>
+            </command_interface>
+            <state_interface name="position"/>
+            <state_interface name="velocity"/>
+            <state_interface name="effort"/>
+        </joint>
     </ros2_control>
 </robot>

File: urdf/robot_description.urdf.xacro (robot description, xacro)
@@ -325,5 +325,5 @@
             <origin xyz="0 0 0" rpy="0 -${pi/2} 0"/>
             <geometry>
-                <mesh filename="$(find custom_robot_sim)/meshes/gripper_finger_mesh.stl" scale="0.002 0.0005 0.01"/>
+                <mesh filename="$(find custom_robot_sim)/meshes/gripper_finger_mesh.stl" scale="0.002 0.0005 0.005"/>
             </geometry>
         </visual>
@@ -347,5 +347,5 @@
     <!-- ==================================== -->
     <joint type="prismatic" name="gripper_finger_right_joint">
-        <mimic joint="gripper_finger_left.joint"/>
+        <mimic joint="gripper_finger_left_joint"/>
         <origin xyz="0.05 0.0 0.055" rpy="0 ${pi/2} ${pi}"/>
         <child link="gripper_finger_right_link"/>
@@ -359,9 +359,9 @@
             <origin xyz="0 0 0" rpy="0 -${pi/2} 0"/>
             <geometry>
-                <mesh filename="$(find custom_robot_sim)/meshes/gripper_finger_mesh.stl" scale="0.002 0.0005 0.01"/>
-            </geometry>
-        </visual>
-        <collision>
-            <origin xyz="-${0.7/2+0.005} 0 -0.035*2" rpy="0 0 0"/>
+                <mesh filename="$(find custom_robot_sim)/meshes/gripper_finger_mesh.stl" scale="0.002 0.0005 0.005"/>
+            </geometry>
+        </visual>
+        <collision>
+            <origin xyz="-${0.7/2+0.005} 0 ${-0.035*2}" rpy="0 0 0"/>
             <geometry>
                 <box size="0.7 0.0375 0.06" />
